File: digits.brd (EAGLE design)
At the start: 160 x 100 mm, 35 parts, among them IC1 STP16CP05 / STP16CPC26, IC2 STP16CP05 / STP16CPC26, IC3 ATMEGA32U4QFN, IC4 ATMEGA32U4TQFP-44, Q1 AO7801, Q2 AO7801, Q3 AO7801

Commit message: added arduinos, layout
Parts:
- removed U$2, U$3, U$4, U$5: BL-S230X-12, digits:BL-S230X-12
- removed U$6: CRYSTALHC49, digits:HC49
- added JP3: M10X2, SparkFun-Connectors:2X10
- added LED1: DEBUG, adafruit:CHIP-LED0805
- added PCB1: ARDUINO_UNO, E14_Arduino:ARDUINO_UNO
- added R8: 910R, SparkFun-Resistors:0805
- added SC1: SPARK_CORECORE, Spark:SPARK_CORE
- added SEG1, SEG2, SEG3, SEG4, SEG5: BL-S230X-12, digits:BL-S230X-12
- added X1: CRYSTALHC49, digits:HC49
- added _1: TEENSY, teensy:TEENSY
- F1: value FUSEMSMF050 -> MF-MSMF075
- JP1: value (none) -> ICSP
- R1: value (none) -> 390R
- R2: value (none) -> 910R
- U$1: value BL-S230X-12 -> TEENSY_30MOD; device digits:BL-S230X-12 -> digits:TEENSY_30_MOD
- moved Q3 334.8 mm to (208.5, -6.15), flipped to the bottom
- moved C2 311.1 mm to (191.4, 37.4), flipped to the bottom, turned to 90 degrees
- moved R2 310.3 mm to (196.0, 29.0), flipped to the bottom, turned to 180 degrees
- moved R7 282.1 mm to (87.2, -32.2), flipped to the bottom, turned to 90 degrees
- moved Q2 280.0 mm to (157.3, -5.15), flipped to the bottom
- moved C9 280.0 mm to (93.0, -37.2), flipped to the bottom, turned to 180 degrees
- moved C7 272.1 mm to (93.0, -43.2), flipped to the bottom, turned to 180 degrees
- moved C8 271.1 mm to (88.2, -51.0), flipped to the bottom, turned to 270 degrees
- moved R6 265.0 mm to (74.5, -48.2), flipped to the bottom
- moved C6 257.8 mm to (82.5, -51.0), flipped to the bottom, turned to 270 degrees
- moved IC2 248.2 mm to (134.1, 35.8), flipped to the bottom, turned to 270 degrees
- moved R5 240.6 mm to (73.0, -41.5), flipped to the bottom, turned to 90 degrees
- moved C5 238.9 mm to (67.5, -50.0), flipped to the bottom, turned to 180 degrees
- moved L1 236.1 mm to (93.0, -47.2), flipped to the bottom
- moved C3 232.2 mm to (93.0, -45.2), flipped to the bottom, turned to 180 degrees
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Connections:
- removed net CLK: IC2.3
- removed net PA0: Q1.2
- removed net PA1: Q1.5
- removed net PA2: Q2.2
- removed net PA3: Q2.5
- removed net PA4: Q3.2
- removed net VBUS: F1.P$2, IC3.7, IC4.7
- new net 3.3V: U$1.3.3V
- new net ARDUINO_VBUS_IN: PCB1.VIN
- new net DEBUG: IC3.22, IC4.22, LED1.A
- new net MAIN_VBUS_IN: F1.P$2
- new net N$10: JP3.5
- new net N$11: JP3.7
- new net N$12: JP3.9
- new net N$13: JP3.11
- new net N$14: JP3.13
- new net N$15: JP3.15
- new net N$16: JP3.17
- new net N$17: JP3.19
- new net N$18: JP3.2
- new net N$19: JP3.4
- new net N$20: JP3.6
- new net N$21: JP3.8
- new net N$22: JP3.10
- new net N$23: JP3.12
- new net N$24: JP3.14
- new net N$25: JP3.16
- new net N$26: JP3.18
- new net N$27: JP3.20
- new net N$6: JP3.1
- new net N$7: LED1.C, R8.1
- new net N$8: SC1.24
- new net N$9: JP3.3
- new net P0: IC3.29, IC4.29, Q1.2
- new net P1: IC3.30, IC4.30, Q1.5
- new net P2: IC3.12, IC4.12, Q2.2
- new net P3: IC3.26, IC4.26, Q2.5
- new net P4: IC3.32, IC4.32, Q3.2
- new net PB0: IC3.8, IC4.8
- new net PB4: IC3.28, IC4.28
- new net PC6: IC3.31, IC4.31
- new net PC7: SC1.23
- new net PD0: IC3.18, IC4.18
- new net PD1: IC3.19, IC4.19
- new net PD2: IC4.20
- new net PD3: IC4.21
- new net PD4: IC3.25, IC4.25
- new net PD7: IC3.27, IC4.27
- new net PE6: IC3.1, IC4.1
- new net PF4: IC3.39, IC4.39
- new net PF5: IC3.38, IC4.38
- new net PF6: IC3.37, IC4.37
- new net PF7: IC3.36, IC4.36
- new net RX: IC3.20, PCB1.0, SC1.4, U$1.0, _1.D2
- new net SC-A0: SC1.12
- new net SC-A1: SC1.11
- new net SC-A2: SC1.10
- new net SC-A6: SC1.6
- new net SC-A7: SC1.5
- new net SC-D2: SC1.15
- new net SC-D5: SC1.18
- new net SC-D6: SC1.19
- new net SC-D7: SC1.20
- new net SCL: PCB1.SCL, SC1.14, U$1.19/A5, _1.D0
- new net SC_VBUS_IN: SC1.1
- new net SDA: PCB1.SDA, SC1.13, U$1.18/A4, _1.D1
- new net T2_VBUS_IN: _1.+5V, _1.5V2
- new net T3_VBUS_IN: U$1.VIN, U$1.VUSB
- new net TX: IC3.21, PCB1.1, SC1.3, U$1.1, _1.D3
- new net VDDA: SC1.22
- net AREF: now also U$1.AREF
- net BLANK: now also IC3.41, IC4.41, SC1.16, U$1.20/A6, _1.C7
- net COL-A1: now also SEG1.17, SEG2.17, SEG3.17, SEG4.17, SEG5.17; no longer U$1.17, U$2.17, U$3.17, U$4.17, U$5.17
- net COL-A2: now also SEG1.14, SEG2.14, SEG3.14, SEG4.14, SEG5.14; no longer U$1.14, U$2.14, U$3.14, U$4.14, U$5.14
- net COL-B: now also SEG1.13, SEG2.13, SEG3.13, SEG4.13, SEG5.13; no longer U$1.13, U$2.13, U$3.13, U$4.13, U$5.13
- net COL-C: now also SEG1.9, SEG2.9, SEG3.9, SEG4.9, SEG5.9; no longer U$1.9, U$2.9, U$3.9, U$4.9, U$5.9
- net COL-D1: now also SEG1.4, SEG2.4, SEG3.4, SEG4.4, SEG5.4; no longer U$1.4, U$2.4, U$3.4, U$4.4, U$5.4
- net COL-D2: now also SEG1.7, SEG2.7, SEG3.7, SEG4.7, SEG5.7; no longer U$1.7, U$2.7, U$3.7, U$4.7, U$5.7
- net COL-DP: now also SEG1.10, SEG2.10, SEG3.10, SEG4.10, SEG5.10; no longer U$1.10, U$2.10, U$3.10, U$4.10, U$5.10
- net COL-DP2: now also SEG1.20, SEG2.20, SEG3.20, SEG4.20, SEG5.20; no longer U$1.20, U$2.20, U$3.20, U$4.20, U$5.20
- net COL-E: now also SEG1.3, SEG2.3, SEG3.3, SEG4.3, SEG5.3; no longer U$1.3, U$2.3, U$3.3, U$4.3, U$5.3
- net COL-F: now also SEG1.19, SEG2.19, SEG3.19, SEG4.19, SEG5.19; no longer U$1.19, U$2.19, U$3.19, U$4.19, U$5.19
- net COL-G1: now also SEG1.2, SEG2.2, SEG3.2, SEG4.2, SEG5.2; no longer U$1.2, U$2.2, U$3.2, U$4.2, U$5.2
- net COL-G2: now also SEG1.12, SEG2.12, SEG3.12, SEG4.12, SEG5.12; no longer U$1.12, U$2.12, U$3.12, U$4.12, U$5.12
- net COL-H: now also SEG1.18, SEG2.18, SEG3.18, SEG4.18, SEG5.18; no longer U$1.18, U$2.18, U$3.18, U$4.18, U$5.18
- net COL-J: now also SEG1.16, SEG2.16, SEG3.16, SEG4.16, SEG5.16; no longer U$1.16, U$2.16, U$3.16, U$4.16, U$5.16
- net COL-K: now also SEG1.15, SEG2.15, SEG3.15, SEG4.15, SEG5.15; no longer IC1.12, U$1.15, U$2.15, U$3.15, U$4.15, U$5.15
- net COL-L: now also IC1.12, SEG1.8, SEG2.8, SEG3.8, SEG4.8, SEG5.8; no longer U$1.8, U$2.8, U$3.8, U$4.8, U$5.8
- net COL-M: now also SEG1.6, SEG2.6, SEG3.6, SEG4.6, SEG5.6; no longer U$1.6, U$2.6, U$3.6, U$4.6, U$5.6
- net COL-N: now also SEG1.5, SEG2.5, SEG3.5, SEG4.5, SEG5.5; no longer U$1.5, U$2.5, U$3.5, U$4.5, U$5.5
- net GND: now also PCB1.GND, PCB1.GND., PCB1.GND.., R8.2, SC1.2, SC1.21, U$1.AGND, U$1.GND, _1.GND, _1.GRND1
- net LATCH: now also IC3.40, IC4.40, SC1.17, U$1.21/A7, _1.C6
- net MISO: now also SC1.8, U$1.12, _1.B3
- net MOSI: now also SC1.7, U$1.11, _1.B2
- net ROW0: now also SEG1.1, SEG1.11; no longer U$1.1, U$1.11
- net ROW1: now also SEG2.1, SEG2.11; no longer U$2.1, U$2.11
- net ROW2: now also SEG3.1, SEG3.11; no longer U$3.1, U$3.11
- net ROW3: now also SEG4.1, SEG4.11; no longer U$4.1, U$4.11
- net ROW4: now also SEG5.1, SEG5.11; no longer U$5.1, U$5.11
- net SCK: now also IC2.3, SC1.9, U$1.13, _1.B1
- net VCC: now also IC3.7, IC4.7
- net XTAL1: now also X1.2; no longer U$6.2
- net XTAL2: now also X1.1; no longer U$6.1
Routing:
- net COL-DP2: track 0.00 -> 199.2 mm, vias 0 -> 4
- net LATCH: track 0.00 -> 197.9 mm, vias 0 -> 3
- net BLANK: track 0.00 -> 187.5 mm, vias 0 -> 3
- net MOSI: track 0.00 -> 184.8 mm, vias 0 -> 2
- net COL-A1: track 0.00 -> 163.3 mm, vias 0 -> 5
- net COL-A2: track 0.00 -> 162.8 mm, vias 0 -> 5
- net COL-G2: track 0.00 -> 158.0 mm, vias 0 -> 4
- net COL-D2: track 0.00 -> 152.3 mm, vias 0 -> 2
- net COL-F: track 0.00 -> 150.9 mm, vias 0 -> 3
- net COL-H: track 0.00 -> 146.8 mm, vias 0 -> 3
- net COL-J: track 0.00 -> 145.2 mm, vias 0 -> 3
- net COL-K: track 0.00 -> 143.5 mm, vias 0 -> 3
- net COL-B: track 0.00 -> 142.6 mm, vias 0 -> 4
- net COL-C: track 0.00 -> 139.1 mm, vias 0 -> 4
- net COL-DP: track 0.00 -> 133.2 mm, vias 0 -> 1
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Other:
- board size 160 x 100 mm -> 246.4 x 75.9 mm

Commit message: updates
Parts:
- removed U$1: TEENSY_30MOD, digits:TEENSY_30_MOD
- removed _1: TEENSY, teensy:TEENSY
- added JP4: Bluefruit LE, SparkFun-Connectors:1X10_LOCK
Connections:
- removed net 3.3V: U$1.3.3V
- removed net T2_VBUS_IN: _1.+5V, _1.5V2
- removed net T3_VBUS_IN: U$1.VIN, U$1.VUSB
- new net BF_ACT: JP4.6
- new net BF_RDY: JP4.5
- new net BF_REQ: JP4.4
- new net BF_RST: JP4.7
- net AREF: no longer U$1.AREF
- net BLANK: no longer U$1.20/A6, _1.C7
- net GND: now also JP4.9; no longer U$1.AGND, U$1.GND, _1.GND, _1.GRND1
- net LATCH: no longer U$1.21/A7, _1.C6
- net MISO: now also JP4.2; no longer U$1.12, _1.B3
- net MOSI: now also JP4.3; no longer U$1.11, _1.B2
- net RX: no longer U$1.0, _1.D2
- net SCK: now also JP4.1; no longer U$1.13, _1.B1
- net SCL: no longer U$1.19/A5, _1.D0
- net SDA: no longer U$1.18/A4, _1.D1
- net TX: no longer U$1.1, _1.D3
- net VCC: now also JP4.10
Routing:
- net LATCH: track 197.9 -> 0.00 mm, vias 3 -> 0
- net BLANK: track 187.5 -> 0.00 mm, vias 3 -> 0
- net MOSI: track 184.8 -> 0.00 mm, vias 2 -> 0
- net SCK: track 130.8 -> 0.00 mm, vias 3 -> 0
- net MISO: track 65.6 -> 0.00 mm
- net TX: track 62.5 -> 0.00 mm, vias 2 -> 0
- net SDA: track 58.7 -> 0.00 mm, vias 2 -> 0
- net RX: track 57.4 -> 0.00 mm, vias 1 -> 0
- net SCL: track 55.2 -> 0.00 mm, vias 2 -> 0

Commit message: moving things around
Parts:
- removed PCB1: ARDUINO_UNO, E14_Arduino:ARDUINO_UNO
- removed SC1: SPARK_CORECORE, Spark:SPARK_CORE
- added J1: POWER_JACKPTH_LOCK, SparkFun-Connectors:POWER_JACK_PTH_LOCK
- added JP5: Adafruit CC3000 Wifi, SparkFun-Connectors:1X09_LOCK
- added SJ1, SJ3: SOLDERJUMPERTRACE, SparkFun-Passives:SJ_2S-TRACE
- added SJ2: SOLDERJUMPERNO, SparkFun-Passives:SJ_2S-NO
Connections:
- removed net ARDUINO_VBUS_IN: PCB1.VIN
- removed net N$10: JP3.5
- removed net N$11: JP3.7
- removed net N$12: JP3.9
- removed net N$13: JP3.11
- removed net N$14: JP3.13
- removed net N$15: JP3.15
- removed net N$16: JP3.17
- removed net N$17: JP3.19
- removed net N$18: JP3.2
- removed net N$19: JP3.4
- removed net N$20: JP3.6
- removed net N$21: JP3.8
- removed net N$22: JP3.10
- removed net N$23: JP3.12
- removed net N$24: JP3.14
- removed net N$25: JP3.16
- removed net N$26: JP3.18
- removed net N$6: JP3.1
- removed net N$8: SC1.24
- removed net N$9: JP3.3
- removed net PB4: IC3.28, IC4.28
- removed net PC7: SC1.23
- removed net PD7: IC3.27, IC4.27
- removed net RX: IC3.20, PCB1.0, SC1.4
- removed net SC-A0: SC1.12
- removed net SC-A1: SC1.11
- removed net SC-A2: SC1.10
- removed net SC-A6: SC1.6
- removed net SC-A7: SC1.5
- removed net SC-D2: SC1.15
- removed net SC-D5: SC1.18
- removed net SC-D6: SC1.19
- removed net SC-D7: SC1.20
- removed net SCL: PCB1.SCL, SC1.14
- removed net SC_VBUS_IN: SC1.1
- removed net SDA: PCB1.SDA, SC1.13
- removed net TX: IC3.21, PCB1.1, SC1.3
- removed net VDDA: SC1.22
- new net PB5: IC3.29, IC4.29, JP3.15
- new net PB6: IC3.30, IC4.30, JP3.17
- new net VIN: JP3.1, JP3.2
- new net WIFI_CS: IC3.27, IC4.27, JP5.7
- new net WIFI_IRQ: JP5.9, SJ3.2
- new net WIFI_VBEN: IC3.28, IC4.28, JP5.8
- net BF_ACT: now also IC3.26, IC4.26
- net BF_RDY: now also SJ1.2, SJ2.2
- net BF_REQ: now also IC3.12, IC4.12
- net BF_RST: now also IC3.32, IC4.32
- net BLANK: no longer SC1.16
- net GND: now also JP3.5, JP3.6, JP5.1; no longer PCB1.GND, PCB1.GND., PCB1.GND.., SC1.2, SC1.21
- net LATCH: no longer SC1.17
- net MISO: now also JP5.5; no longer SC1.8
- net MOSI: now also JP5.6; no longer SC1.7
- net P0: no longer IC3.29, IC4.29
- net P1: no longer IC3.30, IC4.30
- net P2: no longer IC3.12, IC4.12
- net P3: no longer IC3.26, IC4.26
- net P4: no longer IC3.32, IC4.32
- net PB0: now also JP3.19
- net PC6: now also JP3.13
- net PD0: now also JP3.10
- net PD1: now also JP3.8, SJ2.1
- net PD2: now also IC3.20, JP3.7
- net PD3: now also IC3.21, JP3.9
- net PD4: now also JP3.11
- net PE6: now also SJ1.1, SJ3.1
- net PF4: now also JP3.18
- net PF5: now also JP3.16
- net PF6: now also JP3.14
- net PF7: now also JP3.12
- net SCK: now also JP5.4; no longer SC1.9
- net VCC: now also JP3.3, JP3.4, JP5.3
Routing:
- net COL-DP2: track 199.2 -> 0.00 mm, vias 4 -> 0
- net COL-A1: track 163.3 -> 0.00 mm, vias 5 -> 0
- net COL-A2: track 162.8 -> 0.00 mm, vias 5 -> 0
- net COL-G2: track 158.0 -> 0.00 mm, vias 4 -> 0
- net COL-D2: track 152.3 -> 0.00 mm, vias 2 -> 0
- net COL-F: track 150.9 -> 0.00 mm, vias 3 -> 0
- net COL-H: track 146.8 -> 0.00 mm, vias 3 -> 0
- net COL-J: track 145.2 -> 0.00 mm, vias 3 -> 0
- net COL-K: track 143.5 -> 0.00 mm, vias 3 -> 0
- net COL-B: track 142.6 -> 0.00 mm, vias 4 -> 0
- net COL-C: track 139.1 -> 0.00 mm, vias 4 -> 0
- net COL-DP: track 133.2 -> 0.00 mm, vias 1 -> 0
- net COL-L: track 132.6 -> 0.00 mm, vias 3 -> 0
- net COL-G1: track 58.4 -> 0.00 mm, vias 1 -> 0
- net COL-E: track 57.9 -> 0.00 mm, vias 1 -> 0
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
Commit message: adding bigger header
Parts:
- removed JP3: M10X2, SparkFun-Connectors:2X10
- added U$1: HEADER-M26, digits:2X16
- added U$2: TPS54331, Livestream:SOIC-8-PAD
- moved J1 116.0 mm to (-2.00, 56.2), flipped to the bottom, turned to 90 degrees
- moved C3 94.6 mm to (42.6, 34.8)
- moved C4 94.6 mm to (16.9, 47.6)
- moved C5 94.6 mm to (17.1, 30.0)
- moved C6 94.6 mm to (32.1, 29.0)
- moved C7 94.6 mm to (42.6, 36.8)
- moved C8 94.6 mm to (37.9, 29.0)
- moved C9 94.6 mm to (42.6, 42.8)
- moved IC3 94.6 mm to (32.9, 38.8)
- moved IC4 94.6 mm to (32.9, 38.8)
- moved JP1 94.6 mm to (7.99, 39.1)
- moved L1 94.6 mm to (42.6, 32.8)
- moved LED1 94.6 mm to (25.0, 47.7)
- moved R5 94.6 mm to (22.6, 38.5)
- moved R6 94.6 mm to (24.1, 31.8)
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Connections:
- removed net VIN: JP3.1, JP3.2
- new net VLEDS: Q1.3, Q1.6, Q2.3, Q2.6, Q3.6
- net GND: now also U$1.5, U$1.6; no longer JP3.5, JP3.6
- net N$27: now also U$1.20; no longer JP3.20
- net PB0: now also U$1.19; no longer JP3.19
- net PB5: now also U$1.15; no longer JP3.15
- net PB6: now also U$1.17; no longer JP3.17
- net PC6: now also U$1.13; no longer JP3.13
- net PD0: now also U$1.10; no longer JP3.10
- net PD1: now also U$1.8; no longer JP3.8
- net PD2: now also U$1.7; no longer JP3.7
- net PD3: now also U$1.9; no longer JP3.9
- net PD4: now also U$1.11; no longer JP3.11
- net PF4: now also U$1.18; no longer JP3.18
- net PF5: now also U$1.16; no longer JP3.16
- net PF6: now also U$1.14; no longer JP3.14
- net PF7: now also U$1.12; no longer JP3.12
- net VCC: no longer JP3.3, JP3.4, Q1.3, Q1.6, Q2.3, Q2.6, Q3.6
Other:
- board size 246.4 x 75.9 mm -> 251 x 79 mm

Commit message: layout and some parts change
Parts:
- removed F1: MF-MSMF075, digits:MSMF050
- removed Q1, Q2, Q3: AO7801, digits:SC70-6
- removed R7: 10k, SparkFun-Resistors:0805
- removed U$1: HEADER-M26, digits:2X16
- removed U$2: TPS54331, Livestream:SOIC-8-PAD
- added D1: DIODESOD-123F, digits:SOD-123F
- added J2: HEADER-M26, digits:2X16
- added JP3, JP6: M05X2PTH, SparkFun-Connectors:AVR_ICSP
- added SJ4: SOLDERJUMPERTRACE, SparkFun-Retired:SJ_2S-TRACE
- added T1, T2, T3, T4, T5: (no value), zetex:SOT-23
- moved JP5 177.0 mm to (120.0, 52.8), turned to 270 degrees
- moved SJ2 143.7 mm to (75.2, 42.6), flipped to the bottom, turned to 180 degrees
- moved JP4 136.5 mm to (80.0, 52.8), turned to 270 degrees
- moved SJ3 117.0 mm to (58.2, 19.4), flipped to the bottom, turned to 180 degrees
- moved SJ1 110.9 mm to (58.3, 16.5), flipped to the bottom, turned to 180 degrees
- moved IC1 86.5 mm to (182.8, 50.3)
- moved R8 76.1 mm to (26.1, 49.0), turned to 180 degrees
- moved R1 70.6 mm to (176.8, 42.0)
- moved IC2 66.6 mm to (211.3, 26.9)
- moved C1 61.6 mm to (173.5, 47.8), turned to 270 degrees
- moved JP1 24.9 mm to (28.1, 24.4), turned to 180 degrees
- moved C2 16.8 mm to (202.2, 24.5), turned to 270 degrees
- moved R2 14.3 mm to (205.4, 18.2)
- moved Z2 8.10 mm to (14.6, 15.1), turned to 90 degrees
- moved R3 7.21 mm to (16.9, 16.4)
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Connections:
- removed net BF_ACT: IC3.26, IC4.26, JP4.6
- removed net BF_REQ: IC3.12, IC4.12, JP4.4
- removed net BF_RST: IC3.32, IC4.32, JP4.7
- removed net HWB: IC3.33, IC4.33, R7.1
- removed net MAIN_VBUS_IN: F1.P$2
- removed net N$27: U$1.20
- removed net P0: Q1.2
- removed net P1: Q1.5
- removed net P2: Q2.2
- removed net P3: Q2.5
- removed net P4: Q3.2
- removed net PB5: IC3.29, IC4.29, U$1.15
- removed net PB6: IC3.30, IC4.30, U$1.17
- removed net PC6: IC3.31, IC4.31, U$1.13
- removed net PD4: IC3.25, IC4.25, U$1.11
- removed net PF4: IC3.39, IC4.39, U$1.18
- removed net VLEDS: Q1.3, Q1.6, Q2.3, Q2.6, Q3.6
- removed net WIFI_CS: IC3.27, IC4.27, JP5.7
- removed net WIFI_VBEN: IC3.28, IC4.28, JP5.8
- new net GATE0: IC3.25, IC4.25, T1.3
- new net GATE1: IC3.31, IC4.31, T2.3
- new net GATE2: IC3.29, IC4.29, T3.3
- new net GATE3: IC3.30, IC4.30, T4.3
- new net GATE4: IC3.39, IC4.39, T5.3
- new net N$8: IC3.14, IC3.34
- new net PB4: IC3.28, IC4.28, J2.10, JP5.8
- new net PB7: IC3.12, IC4.12, J2.12, JP4.4
- new net PC7: IC3.32, IC4.32, J2.16, JP4.7
- new net PD6: IC3.26, IC4.26, J2.14, JP4.6
- new net PD7: IC3.27, IC4.27, J2.6, JP5.7
- new net PRESENCE: IC3.33, IC4.33, J2.23
- new net SDO2: IC2.22, JP3.3
- new net VCCIC: C8.1, C9.1, IC3.2, IC3.7, IC4.14, IC4.2, IC4.34, IC4.7, JP1.2, L1.1, R6.2, SJ4.1
- net BLANK: now also J2.21, JP3.6
- net GND: now also J1.GND, J2.25, J2.26, J2.3, J2.4, JP3.10, JP3.9; no longer R7.2, U$1.5, U$1.6
- net LATCH: now also J2.19, JP3.5
- net MISO: now also J2.15
- net MOSI: now also J2.13
- net N$3: now also D1.A; no longer F1.P$1
- net PB0: now also J2.18; no longer U$1.19
- net PD0: now also J2.9, JP3.7; no longer U$1.10
- net PD1: now also J2.11, JP3.8; no longer U$1.8
- net PD2: now also J2.5; no longer U$1.7
- net PD3: now also J2.7; no longer U$1.9
- net PE6: now also J2.8
- net PF5: now also J2.24; no longer U$1.16
- net PF6: now also J2.22; no longer U$1.14
- net PF7: now also J2.20; no longer U$1.12
- net ROW0: now also T1.2; no longer Q1.1
- net ROW1: now also T2.2; no longer Q1.4
- net ROW2: now also T3.2; no longer Q2.1
- net ROW3: now also T4.2; no longer Q2.4
- net ROW4: now also T5.2; no longer Q3.1
- net SCK: now also J2.17, JP3.4
- net VCC: now also D1.C, J1.PWR, J2.1, J2.2, JP3.1, JP3.2, SJ4.2, T1.1, T2.1, T3.1, T4.1, T5.1; no longer C8.1, C9.1, IC3.14, IC3.2, IC3.34, IC3.7, IC4.14, IC4.2, IC4.34, IC4.7, JP1.2, L1.1, R6.2
Routing:
- net VCC: track 0.00 -> 342.2 mm, vias 0 -> 2
- net SCK: track 0.00 -> 219.2 mm, vias 0 -> 3
- net BLANK: track 0.00 -> 200.1 mm, vias 0 -> 4
- net LATCH: track 0.00 -> 194.9 mm, vias 0 -> 5
- net GATE4: track 0.00 -> 194.7 mm, vias 0 -> 2
- net GATE3: track 0.00 -> 163.2 mm, vias 0 -> 2
- net MOSI: track 0.00 -> 134.5 mm, vias 0 -> 5
- net PB0: track 0.00 -> 118.4 mm, vias 0 -> 3
- net GATE2: track 0.00 -> 116.2 mm, vias 0 -> 2
- net MISO: track 0.00 -> 112.1 mm, vias 0 -> 2
- net PB7: track 0.00 -> 111.9 mm, vias 0 -> 4
- net COL-DP2: track 0.00 -> 108.6 mm, vias 0 -> 3
- net COL-DP: track 0.00 -> 102.4 mm
- net COL-A2: track 0.00 -> 95.9 mm, vias 0 -> 1
- net COL-A1: track 0.00 -> 94.8 mm, vias 0 -> 1
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- added copper zone on layer 1, net GND

Commit message: layout
Parts:
- moved JP6 255.5 mm to (236.1, 38.5), turned to 180 degrees
- moved JP2 5.80 mm to (8.39, 17.7)
- moved JP3 3.13 mm to (7.00, 37.5)
- moved SJ2 1.20 mm to (76.4, 42.7)
- moved Z1 0.30 mm to (14.6, 19.2)
- moved Z2 0.20 mm to (14.6, 15.3)
- flipped J2 to the bottom
- flipped JP4 to the bottom
- flipped JP5 to the bottom
Connections:
- net BLANK: now also JP6.5
- net GND: now also JP6.1, JP6.2
- net LATCH: now also JP6.6
- net MOSI: now also JP3.3
- net PD0: now also JP6.4
- net PD1: now also JP6.3
- net SCK: now also JP6.7
- net SDO2: now also JP6.8; no longer JP3.3
- net VCC: now also JP6.10, JP6.9
Routing:
- net LATCH: track 194.9 -> 377.4 mm, vias 5 -> 7
- net BLANK: track 200.1 -> 381.5 mm, vias 4 -> 5
- net PB4: track 47.9 -> 105.6 mm
- net PD7: track 46.7 -> 104.1 mm, vias 0 -> 1
- net PD1: track 69.4 -> 107.7 mm, vias 1 -> 2
- net PD0: track 70.5 -> 103.0 mm, vias 1 -> 4
- net MOSI: track 134.5 -> 166.8 mm, vias 5 -> 8
- net MISO: track 112.1 -> 143.1 mm, vias 2 -> 3
- net VCCIC: track 48.5 -> 73.1 mm, vias 3 -> 5
- net GND: track 14.0 -> 38.4 mm, vias 0 -> 10
- net SCK: track 219.2 -> 242.9 mm, vias 3 -> 7
- net PE6: track 44.6 -> 65.9 mm, vias 2 -> 3
- net PB7: track 111.9 -> 125.2 mm
- net PD6: track 57.6 -> 70.0 mm, vias 2 -> 3
- net PC7: track 46.5 -> 58.6 mm
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Other:
- board size 251 x 79 mm -> 240.9 x 79 mm

Commit message: more layout
Parts:
- JP3, JP6: value M05X2PTH -> M05X2SHD; device SparkFun-Connectors:AVR_ICSP -> SparkFun-Connectors:2X5-SHROUDED
- moved IC2 41.3 mm to (170.0, 28.2)
- moved C2 38.6 mm to (163.8, 20.5), turned to 0 degrees
- moved R2 38.4 mm to (167.1, 20.5), turned to 0 degrees
- moved JP6 36.1 mm to (200.0, 37.5), flipped to the bottom
- moved IC1 13.2 mm to (170.0, 47.2)
- moved R1 12.5 mm to (164.8, 38.6), turned to 90 degrees
- moved C1 12.2 mm to (161.4, 45.9), turned to 90 degrees
- moved T3 2.21 mm to (105.8, 4.30), turned to 0 degrees
- moved T5 2.15 mm to (202.6, 4.50), turned to 0 degrees
- moved T1 2.12 mm to (9.40, 4.40), turned to 0 degrees
- moved T2 2.00 mm to (57.1, 4.40), turned to 0 degrees
- moved T4 1.96 mm to (154.0, 4.50), turned to 0 degrees
- flipped JP3 to the bottom
Routing:
- net COL-E: track 0.00 -> 297.9 mm, vias 0 -> 7
- net COL-N: track 0.00 -> 277.4 mm, vias 0 -> 7
- net COL-C: track 0.00 -> 273.7 mm, vias 0 -> 7
- net COL-M: track 0.00 -> 270.1 mm, vias 0 -> 7
- net COL-L: track 0.00 -> 268.4 mm, vias 0 -> 7
- net VCC: track 335.8 -> 588.6 mm, vias 2 -> 9
- net COL-D2: track 32.0 -> 256.7 mm, vias 0 -> 5
- net COL-G1: track 37.2 -> 257.1 mm, vias 2 -> 7
- net COL-D1: track 37.1 -> 254.3 mm, vias 0 -> 5
- net COL-A2: track 95.9 -> 284.1 mm, vias 1 -> 4
- net COL-G2: track 93.4 -> 281.2 mm, vias 0 -> 4
- net COL-A1: track 94.8 -> 282.1 mm, vias 1 -> 4
- net PD0: track 103.0 -> 268.8 mm, vias 4 -> 7
- net COL-DP2: track 108.6 -> 274.2 mm, vias 3 -> 5
- net COL-K: track 64.9 -> 225.4 mm, vias 0 -> 5
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
Commit message: layout and working on silks
Parts:
- J2: value HEADER-M26 -> ACCESSORY
- moved SJ1 17.3 mm to (75.1, 20.7)
- moved SJ3 17.0 mm to (75.1, 17.9)
- moved D1 1.58 mm to (6.40, 9.70), turned to 180 degrees
Connections:
- removed net N$8: IC3.14, IC3.34
- net VCCIC: now also IC3.14, IC3.34
Routing:
- net ROW3: track 2.56 -> 99.0 mm, vias 0 -> 4
- net ROW0: track 2.38 -> 97.1 mm, vias 0 -> 2
- net ROW1: track 2.94 -> 94.8 mm, vias 0 -> 3
- net ROW2: track 2.54 -> 94.0 mm, vias 0 -> 3
- net ROW4: track 2.22 -> 87.2 mm, vias 0 -> 2
- net VCC: track 588.6 -> 665.9 mm, vias 9 -> 8
- net WIFI_IRQ: track 0.00 -> 59.3 mm, vias 0 -> 1
- net BLANK: track 303.3 -> 337.4 mm, vias 5 -> 6
- net LATCH: track 271.5 -> 305.5 mm, vias 5 -> 6
- net BF_RDY: track 3.05 -> 27.4 mm, vias 0 -> 1
- net PE6: track 65.9 -> 84.6 mm
- net N$3: track 0.00 -> 12.0 mm
- net VCCIC: track 73.1 -> 81.7 mm, vias 5 -> 6
- net GND: track 48.1 -> 56.6 mm, vias 16 -> 19
- net AVCC: track 36.0 -> 37.7 mm
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