File: digits.sch (EAGLE design)
At the start: 35 parts, among them IC1 STP16CP05 / STP16CPC26, IC2 STP16CP05 / STP16CPC26, IC3 ATMEGA32U4QFN, IC4 ATMEGA32U4TQFP-44, Q1 AO7801, Q2 AO7801, Q3 AO7801

Commit message: added arduinos, layout
Parts:
- added JP3: M10X2, SparkFun-Connectors:M10X2
- added LED1: DEBUG, adafruit:LEDCHIP-LED0805
- added PCB1: ARDUINO_UNO, E14_Arduino:ARDUINO_UNO
- added R8: 910R, SparkFun-Resistors:RESISTOR0805-RES
- added SC1: SPARK_CORECORE, Spark:SPARK_CORECORE
- added SEG1: BL-S230X-12, digits:BL-S230X-12
- added _1: TEENSY, teensy:TEENSY
- F1: value FUSEMSMF050 -> MF-MSMF075
- JP1: value (none) -> ICSP
- R1: value (none) -> 390R
- R2: value (none) -> 910R
- U$1: value BL-S230X-12 -> TEENSY_30MOD; device digits:BL-S230X-12 -> digits:TEENSY_30MOD
- renumbered U$2 to SEG2, U$3 to SEG3, U$4 to SEG4, U$5 to SEG5, U$6 to X1
Connections:
- removed net CLK: IC2.CLK
- removed net PA0: Q1.G1
- removed net PA1: Q1.G2
- removed net PA2: Q2.G1
- removed net PA3: Q2.G2
- removed net PA4: Q3.G1
- removed net VBUS: F1.2, IC3.VBUS, IC4.VBUS
- new net ARDUINO_VBUS_IN: PCB1.VIN
- new net DEBUG: IC3.PD5, IC4.PD5, LED1.A
- new net MAIN_VBUS_IN: F1.2
- new net N$10: JP3.5
- new net N$11: JP3.7
- new net N$12: JP3.9
- new net N$13: JP3.11
- new net N$14: JP3.13
- new net N$15: JP3.15
- new net N$16: JP3.17
- new net N$17: JP3.19
- new net N$18: JP3.2
- new net N$19: JP3.4
- new net N$20: JP3.6
- new net N$21: JP3.8
- new net N$22: JP3.10
- new net N$23: JP3.12
- new net N$24: JP3.14
- new net N$25: JP3.16
- new net N$26: JP3.18
- new net N$27: JP3.20
- new net N$6: JP3.1
- new net N$7: LED1.C, R8.1
- new net N$8: SC1.VCC
- new net N$9: JP3.3
- new net P0: IC3.PB5(ADC12), IC4.PB5(ADC12), Q1.G1
- new net P1: IC3.PB6(ADC13), IC4.PB6(ADC13), Q1.G2
- new net P2: IC3.PB7, IC4.PB7, Q2.G1
- new net P3: IC3.PD6(ADC9), IC4.PD6(ADC9), Q2.G2
- new net P4: IC3.PC7, IC4.PC7, Q3.G1
- new net PB0: IC3.PB0(SS), IC4.PB0(SS)
- new net PB4: IC3.PB4(ADC11), IC4.PB4(ADC11)
- new net PC6: IC3.PC6, IC4.PC6
- new net PC7: SC1.!RST
- new net PD0: IC3.PD0(SCL), IC4.PD0(SCL)
- new net PD1: IC3.PD1(SDA), IC4.PD1(SDA)
- new net PD2: IC4.PD2(RX)
- new net PD3: IC4.PD3(TX)
- new net PD4: IC3.PD4(ADC8), IC4.PD4(ADC8)
- new net PD7: IC3.PD7(ADC10), IC4.PD7(ADC10)
- new net PE6: IC3.PE6, IC4.PE6
- new net PF4: IC3.PF4(ADC4), IC4.PF4(ADC4)
- new net PF5: IC3.PF5(ADC5), IC4.PF5(ADC5)
- new net PF6: IC3.PF6(ADC6), IC4.PF6(ADC6)
- new net PF7: IC3.PF7(ADC7), IC4.PF7(ADC7)
- new net RX: IC3.PD2(RX), PCB1.0(RX), SC1.RX, U$1.0, _1._D2
- new net SC-A0: SC1.A0
- new net SC-A1: SC1.A1
- new net SC-A2: SC1.A2
- new net SC-A6: SC1.A6
- new net SC-A7: SC1.A7
- new net SC-D2: SC1.D2
- new net SC-D5: SC1.D5
- new net SC-D6: SC1.D6
- new net SC-D7: SC1.D7
- new net SCL: PCB1.28(SCL), SC1.D1, U$1.19/A5, _1._D0
- new net SC_VBUS_IN: SC1.RAW
- new net SDA: PCB1.27(SDA), SC1.D0, U$1.18/A4, _1._D1
- new net T2_VBUS_IN: _1.5V, _1._5V2
- new net T3_VBUS_IN: U$1.VIN, U$1.VUSB
- new net TX: IC3.PD3(TX), PCB1.1(TX), SC1.TX, U$1.1, _1._D3
- net BLANK: now also IC3.PF0(ADC0), IC4.PF0(ADC0), SC1.D3, U$1.20/A6, _1._C7
- net COL-A1: now also SEG1.A1; no longer U$1.A1
- net COL-A2: now also SEG1.A2; no longer U$1.A2
- net COL-B: now also SEG1.B; no longer U$1.B
- net COL-C: now also SEG1.C; no longer U$1.C
- net COL-D1: now also SEG1.D1; no longer U$1.D1
- net COL-D2: now also SEG1.D2; no longer U$1.D2
- net COL-DP: now also SEG1.DP; no longer U$1.DP
- net COL-DP2: now also SEG1.DP2; no longer U$1.DP2
- net COL-E: now also SEG1.E; no longer U$1.E
- net COL-F: now also SEG1.F; no longer U$1.F
- net COL-G1: now also SEG1.G1; no longer U$1.G1
- net COL-G2: now also SEG1.G2; no longer U$1.G2
- net COL-H: now also SEG1.H; no longer U$1.H
- net COL-J: now also SEG1.J; no longer U$1.J
- net COL-K: now also SEG1.K; no longer IC1.OUT7, U$1.K
- net COL-L: now also IC1.OUT7, SEG1.L; no longer U$1.L
- net COL-M: now also SEG1.M; no longer U$1.M
- net COL-N: now also SEG1.N; no longer U$1.N
- net GND: now also PCB1.GND, PCB1.GND., PCB1.GND.., R8.2, SC1.GND@2, SC1.GND@21, U$1.AGND, U$1.GND, _1._GND, _1._GND1
- net LATCH: now also IC3.PF1(ADC1), IC4.PF1(ADC1), SC1.D4, U$1.21/A7, _1._C6
- net MISO: now also SC1.A4, U$1.12, _1._B3
- net MOSI: now also SC1.A5, U$1.11, _1._B2
- net ROW0: now also SEG1.COM; no longer U$1.COM
- net SCK: now also IC2.CLK, SC1.A3, U$1.13, _1._B1
- net VCC: now also IC3.VBUS, IC4.VBUS

Commit message: updates
Parts:
- removed U$1: TEENSY_30MOD, digits:TEENSY_30MOD
- removed _1: TEENSY, teensy:TEENSY
- added JP4: Bluefruit LE, SparkFun-Connectors:M10LOCK
Connections:
- removed net T2_VBUS_IN: _1.5V, _1._5V2
- removed net T3_VBUS_IN: U$1.VIN, U$1.VUSB
- new net BF_ACT: JP4.6
- new net BF_RDY: JP4.5
- new net BF_REQ: JP4.4
- new net BF_RST: JP4.7
- net BLANK: no longer U$1.20/A6, _1._C7
- net GND: now also JP4.9; no longer U$1.AGND, U$1.GND, _1._GND, _1._GND1
- net LATCH: no longer U$1.21/A7, _1._C6
- net MISO: now also JP4.2; no longer U$1.12, _1._B3
- net MOSI: now also JP4.3; no longer U$1.11, _1._B2
- net RX: no longer U$1.0, _1._D2
- net SCK: now also JP4.1; no longer U$1.13, _1._B1
- net SCL: no longer U$1.19/A5, _1._D0
- net SDA: no longer U$1.18/A4, _1._D1
- net TX: no longer U$1.1, _1._D3
- net VCC: now also JP4.10

Commit message: moving things around
Parts:
- removed PCB1: ARDUINO_UNO, E14_Arduino:ARDUINO_UNO
- removed SC1: SPARK_CORECORE, Spark:SPARK_CORECORE
- added J1: POWER_JACKPTH_LOCK, SparkFun-Connectors:POWER_JACKPTH_LOCK
- added JP5: Adafruit CC3000 Wifi, SparkFun-Connectors:M09LOCK
- added SJ1, SJ3: SOLDERJUMPERTRACE, SparkFun-Passives:SOLDERJUMPERTRACE
- added SJ2: SOLDERJUMPERNO, SparkFun-Passives:SOLDERJUMPERNO
Connections:
- removed net ARDUINO_VBUS_IN: PCB1.VIN
- removed net N$10: JP3.5
- removed net N$11: JP3.7
- removed net N$12: JP3.9
- removed net N$13: JP3.11
- removed net N$14: JP3.13
- removed net N$15: JP3.15
- removed net N$16: JP3.17
- removed net N$17: JP3.19
- removed net N$18: JP3.2
- removed net N$19: JP3.4
- removed net N$20: JP3.6
- removed net N$21: JP3.8
- removed net N$22: JP3.10
- removed net N$23: JP3.12
- removed net N$24: JP3.14
- removed net N$25: JP3.16
- removed net N$26: JP3.18
- removed net N$6: JP3.1
- removed net N$8: SC1.VCC
- removed net N$9: JP3.3
- removed net PB4: IC3.PB4(ADC11), IC4.PB4(ADC11)
- removed net PC7: SC1.!RST
- removed net PD7: IC3.PD7(ADC10), IC4.PD7(ADC10)
- removed net RX: IC3.PD2(RX), PCB1.0(RX), SC1.RX
- removed net SC-A0: SC1.A0
- removed net SC-A1: SC1.A1
- removed net SC-A2: SC1.A2
- removed net SC-A6: SC1.A6
- removed net SC-A7: SC1.A7
- removed net SC-D2: SC1.D2
- removed net SC-D5: SC1.D5
- removed net SC-D6: SC1.D6
- removed net SC-D7: SC1.D7
- removed net SCL: PCB1.28(SCL), SC1.D1
- removed net SC_VBUS_IN: SC1.RAW
- removed net SDA: PCB1.27(SDA), SC1.D0
- removed net TX: IC3.PD3(TX), PCB1.1(TX), SC1.TX
- new net PB5: IC3.PB5(ADC12), IC4.PB5(ADC12), JP3.15
- new net PB6: IC3.PB6(ADC13), IC4.PB6(ADC13), JP3.17
- new net VIN: JP3.1, JP3.2
- new net WIFI_CS: IC3.PD7(ADC10), IC4.PD7(ADC10), JP5.7
- new net WIFI_IRQ: JP5.9, SJ3.2
- new net WIFI_VBEN: IC3.PB4(ADC11), IC4.PB4(ADC11), JP5.8
- net BF_ACT: now also IC3.PD6(ADC9), IC4.PD6(ADC9)
- net BF_RDY: now also SJ1.2, SJ2.2
- net BF_REQ: now also IC3.PB7, IC4.PB7
- net BF_RST: now also IC3.PC7, IC4.PC7
- net BLANK: no longer SC1.D3
- net GND: now also JP3.5, JP3.6, JP5.1; no longer PCB1.GND, PCB1.GND., PCB1.GND.., SC1.GND@2, SC1.GND@21
- net LATCH: no longer SC1.D4
- net MISO: now also JP5.5; no longer SC1.A4
- net MOSI: now also JP5.6; no longer SC1.A5
- net P0: no longer IC3.PB5(ADC12), IC4.PB5(ADC12)
- net P1: no longer IC3.PB6(ADC13), IC4.PB6(ADC13)
- net P2: no longer IC3.PB7, IC4.PB7
- net P3: no longer IC3.PD6(ADC9), IC4.PD6(ADC9)
- net P4: no longer IC3.PC7, IC4.PC7
- net PB0: now also JP3.19
- net PC6: now also JP3.13
- net PD0: now also JP3.10
- net PD1: now also JP3.8, SJ2.1
- net PD2: now also IC3.PD2(RX), JP3.7
- net PD3: now also IC3.PD3(TX), JP3.9
- net PD4: now also JP3.11
- net PE6: now also SJ1.1, SJ3.1
- net PF4: now also JP3.18
- net PF5: now also JP3.16
- net PF6: now also JP3.14
- net PF7: now also JP3.12
- net SCK: now also JP5.4; no longer SC1.A3
- net VCC: now also JP3.3, JP3.4, JP5.3
Other:
- moved on the sheet: JP3, JP4

Commit message: adding bigger header
Parts:
- removed JP3: M10X2, SparkFun-Connectors:M10X2
- added U$1: HEADER-M26, digits:HEADER-M26
- added U$2: TPS54331, Livestream:TPS54331
Connections:
- removed net VIN: JP3.1, JP3.2
- new net VLEDS: Q1.D1, Q1.D2, Q2.D1, Q2.D2, Q3.D1
- net GND: now also U$1.5, U$1.6; no longer JP3.5, JP3.6
- net N$27: now also U$1.20; no longer JP3.20
- net PB0: now also U$1.19; no longer JP3.19
- net PB5: now also U$1.15; no longer JP3.15
- net PB6: now also U$1.17; no longer JP3.17
- net PC6: now also U$1.13; no longer JP3.13
- net PD0: now also U$1.10; no longer JP3.10
- net PD1: now also U$1.8; no longer JP3.8
- net PD2: now also U$1.7; no longer JP3.7
- net PD3: now also U$1.9; no longer JP3.9
- net PD4: now also U$1.11; no longer JP3.11
- net PF4: now also U$1.18; no longer JP3.18
- net PF5: now also U$1.16; no longer JP3.16
- net PF6: now also U$1.14; no longer JP3.14
- net PF7: now also U$1.12; no longer JP3.12
- net VCC: no longer JP3.3, JP3.4, Q1.D1, Q1.D2, Q2.D1, Q2.D2, Q3.D1

Commit message: layout and some parts change
Parts:
- removed F1: MF-MSMF075, digits:FUSEMSMF050
- removed Q1, Q2, Q3: AO7801, digits:AO7801
- removed R7: 10k, SparkFun-Resistors:RESISTOR0805-RES
- removed U$1: HEADER-M26, digits:HEADER-M26
- removed U$2: TPS54331, Livestream:TPS54331
- added D1: DIODESOD-123F, digits:DIODESOD-123F
- added J2: HEADER-M26, digits:HEADER-M26
- added JP3, JP6: M05X2PTH, SparkFun-Connectors:M05X2PTH
- added SJ4: SOLDERJUMPERTRACE, SparkFun-Retired:SOLDERJUMPERTRACE
- added T1, T2, T3, T4, T5: (no value), zetex:PMOSSOT23
Connections:
- removed net BF_ACT: IC3.PD6(ADC9), IC4.PD6(ADC9), JP4.6
- removed net BF_REQ: IC3.PB7, IC4.PB7, JP4.4
- removed net BF_RST: IC3.PC7, IC4.PC7, JP4.7
- removed net HWB: IC3.PE2/!HWB, IC4.PE2/!HWB, R7.1
- removed net MAIN_VBUS_IN: F1.2
- removed net N$27: U$1.20
- removed net P0: Q1.G1
- removed net P1: Q1.G2
- removed net P2: Q2.G1
- removed net P3: Q2.G2
- removed net P4: Q3.G1
- removed net PB5: IC3.PB5(ADC12), IC4.PB5(ADC12), U$1.15
- removed net PB6: IC3.PB6(ADC13), IC4.PB6(ADC13), U$1.17
- removed net PC6: IC3.PC6, IC4.PC6, U$1.13
- removed net PD4: IC3.PD4(ADC8), IC4.PD4(ADC8), U$1.11
- removed net PF4: IC3.PF4(ADC4), IC4.PF4(ADC4), U$1.18
- removed net VLEDS: Q1.D1, Q1.D2, Q2.D1, Q2.D2, Q3.D1
- removed net WIFI_CS: IC3.PD7(ADC10), IC4.PD7(ADC10), JP5.7
- removed net WIFI_VBEN: IC3.PB4(ADC11), IC4.PB4(ADC11), JP5.8
- new net GATE0: IC3.PD4(ADC8), IC4.PD4(ADC8), T1.G
- new net GATE1: IC3.PC6, IC4.PC6, T2.G
- new net GATE2: IC3.PB5(ADC12), IC4.PB5(ADC12), T3.G
- new net GATE3: IC3.PB6(ADC13), IC4.PB6(ADC13), T4.G
- new net GATE4: IC3.PF4(ADC4), IC4.PF4(ADC4), T5.G
- new net N$8: IC3.VCC@14, IC3.VCC@34
- new net PB4: IC3.PB4(ADC11), IC4.PB4(ADC11), J2.10, JP5.8
- new net PB7: IC3.PB7, IC4.PB7, J2.12, JP4.4
- new net PC7: IC3.PC7, IC4.PC7, J2.16, JP4.7
- new net PD6: IC3.PD6(ADC9), IC4.PD6(ADC9), J2.14, JP4.6
- new net PD7: IC3.PD7(ADC10), IC4.PD7(ADC10), J2.6, JP5.7
- new net PRESENCE: IC3.PE2/!HWB, IC4.PE2/!HWB, J2.23
- new net SDO2: IC2.SDO, JP3.3
- new net VCCIC: C8.1, C9.1, IC3.UVCC, IC3.VBUS, IC4.UVCC, IC4.VBUS, IC4.VCC@14, IC4.VCC@34, JP1.2, L1.1, R6.2, SJ4.1
- net BLANK: now also J2.21, JP3.6
- net GND: now also J1.GND, J2.25, J2.26, J2.3, J2.4, JP3.10, JP3.9; no longer R7.2, U$1.5, U$1.6
- net LATCH: now also J2.19, JP3.5
- net MISO: now also J2.15
- net MOSI: now also J2.13
- net N$3: now also D1.A; no longer F1.1
- net PB0: now also J2.18; no longer U$1.19
- net PD0: now also J2.9, JP3.7; no longer U$1.10
- net PD1: now also J2.11, JP3.8; no longer U$1.8
- net PD2: now also J2.5; no longer U$1.7
- net PD3: now also J2.7; no longer U$1.9
- net PE6: now also J2.8
- net PF5: now also J2.24; no longer U$1.16
- net PF6: now also J2.22; no longer U$1.14
- net PF7: now also J2.20; no longer U$1.12
- net ROW0: now also T1.S; no longer Q1.S1
- net ROW1: now also T2.S; no longer Q1.S2
- net ROW2: now also T3.S; no longer Q2.S1
- net ROW3: now also T4.S; no longer Q2.S2
- net ROW4: now also T5.S; no longer Q3.S1
- net SCK: now also J2.17, JP3.4
- net VCC: now also D1.C, J1.PWR, J2.1, J2.2, JP3.1, JP3.2, SJ4.2, T1.D, T2.D, T3.D, T4.D, T5.D; no longer C8.1, C9.1, IC3.UVCC, IC3.VBUS, IC3.VCC@14, IC3.VCC@34, IC4.UVCC, IC4.VBUS, IC4.VCC@14, IC4.VCC@34, JP1.2, L1.1, R6.2
Other:
- moved on the sheet: J1, JP4, JP5, R6

Commit message: layout
Connections:
- net BLANK: now also JP6.5
- net GND: now also JP6.1, JP6.2
- net LATCH: now also JP6.6
- net MOSI: now also JP3.3
- net PD0: now also JP6.4
- net PD1: now also JP6.3
- net SCK: now also JP6.7
- net SDO2: now also JP6.8; no longer JP3.3
- net VCC: now also JP6.10, JP6.9
Other:
- moved on the sheet: JP6
Changed lines of the file:
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@@
 <instance part="SUPPLY3" gate="G$1" x="254" y="45.72"/>
 <instance part="JP3" gate="G$1" x="12.7" y="38.1"/>
-<instance part="JP6" gate="G$1" x="96.52" y="38.1"/>
+<instance part="JP6" gate="G$1" x="53.34" y="38.1" rot="R180"/>
 <instance part="SJ4" gate="1" x="279.4" y="73.66" rot="R90"/>
 <instance part="SUPPLY4" gate="G$1" x="279.4" y="83.82"/>
@@
 <pinref part="SJ4" gate="1" pin="2"/>
 <wire x1="279.4" y1="83.82" x2="279.4" y2="78.74" width="0.1524" layer="91"/>
+</segment>
+<segment>
+<pinref part="JP6" gate="G$1" pin="10"/>
+<wire x1="45.72" y1="43.18" x2="43.18" y2="43.18" width="0.1524" layer="91"/>
+<label x="43.18" y="43.18" size="1.4224" layer="95" rot="R180" xref="yes"/>
+</segment>
+<segment>
+<pinref part="JP6" gate="G$1" pin="9"/>
+<wire x1="60.96" y1="43.18" x2="63.5" y2="43.18" width="0.1524" layer="91"/>
+<label x="63.5" y="43.18" size="1.4224" layer="95" xref="yes"/>
 </segment>
 </net>
@@
 <label x="22.86" y="33.02" size="1.4224" layer="95" xref="yes"/>
 </segment>
+<segment>
+<pinref part="JP6" gate="G$1" pin="2"/>
+<wire x1="45.72" y1="33.02" x2="43.18" y2="33.02" width="0.1524" layer="91"/>
+<label x="43.18" y="33.02" size="1.4224" layer="95" rot="R180" xref="yes"/>
+</segment>
+<segment>
+<pinref part="JP6" gate="G$1" pin="1"/>
+<wire x1="60.96" y1="33.02" x2="63.5" y2="33.02" width="0.1524" layer="91"/>
+<label x="63.5" y="33.02" size="1.4224" layer="95" xref="yes"/>
+</segment>
 </net>
 <net name="N$1" class="0">
@@
 <pinref part="J2" gate="G$1" pin="13"/>
 </segment>
+<segment>
+<pinref part="JP3" gate="G$1" pin="3"/>
+<wire x1="5.08" y1="40.64" x2="2.54" y2="40.64" width="0.1524" layer="91"/>
+<label x="2.54" y="40.64" size="1.4224" layer="95" rot="R180" xref="yes"/>
+</segment>
 </net>
 <net name="SCK" class="0">
@@
 <label x="22.86" y="40.64" size="1.4224" layer="95" xref="yes"/>
 </segment>
+<segment>
+<pinref part="JP6" gate="G$1" pin="7"/>
+<wire x1="60.96" y1="40.64" x2="63.5" y2="40.64" width="0.1524" layer="91"/>
+<label x="63.5" y="40.64" size="1.4224" layer="95" xref="yes"/>
+</segment>
 </net>
 <net name="SDO" class="0">
@@
 <label x="2.54" y="38.1" size="1.4224" layer="95" rot="R180" xref="yes"/>
 </segment>
+<segment>
+<pinref part="JP6" gate="G$1" pin="6"/>
+<wire x1="45.72" y1="38.1" x2="43.18" y2="38.1" width="0.1524" layer="91"/>
+<label x="43.18" y="38.1" size="1.4224" layer="95" rot="R180" xref="yes"/>
+</segment>
 </net>
 <net name="BLANK" class="0">
@@
 <wire x1="20.32" y1="38.1" x2="22.86" y2="38.1" width="0.1524" layer="91"/>
 <label x="22.86" y="38.1" size="1.4224" layer="95" xref="yes"/>
+</segment>
+<segment>
+<pinref part="JP6" gate="G$1" pin="5"/>
+<wire x1="60.96" y1="38.1" x2="63.5" y2="38.1" width="0.1524" layer="91"/>
+<label x="63.5" y="38.1" size="1.4224" layer="95" xref="yes"/>
 </segment>
 </net>
@@
 <label x="22.86" y="35.56" size="1.4224" layer="95" xref="yes"/>
 </segment>
+<segment>
+<pinref part="JP6" gate="G$1" pin="3"/>
+<wire x1="60.96" y1="35.56" x2="63.5" y2="35.56" width="0.1524" layer="91"/>
+<label x="63.5" y="35.56" size="1.4224" layer="95" xref="yes"/>
+</segment>
 </net>
 <net name="PD0" class="0">
@@
 <label x="2.54" y="35.56" size="1.4224" layer="95" rot="R180" xref="yes"/>
 </segment>
+<segment>
+<pinref part="JP6" gate="G$1" pin="4"/>
+<wire x1="45.72" y1="35.56" x2="43.18" y2="35.56" width="0.1524" layer="91"/>
+<label x="43.18" y="35.56" size="1.4224" layer="95" rot="R180" xref="yes"/>
+</segment>
 </net>
 <net name="PE6" class="0">
@@
 </segment>
 <segment>
-<pinref part="JP3" gate="G$1" pin="3"/>
-<wire x1="5.08" y1="40.64" x2="2.54" y2="40.64" width="0.1524" layer="91"/>
-<label x="2.54" y="40.64" size="1.4224" layer="95" rot="R180" xref="yes"/>
-</segment>
-</net>
+<pinref part="JP6" gate="G$1" pin="8"/>
+<wire x1="45.72" y1="40.64" x2="43.18" y2="40.64" width="0.1524" layer="91"/>
+<label x="43.18" y="40.64" size="1.4224" layer="95" rot="R180" xref="yes"/>
+</segment>
+</net>

Commit message: more layout
Parts:
- JP3, JP6: value M05X2PTH -> M05X2SHD; device SparkFun-Connectors:M05X2PTH -> SparkFun-Connectors:M05X2SHD
Changed lines of the file:
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@@
 <part name="D1" library="digits" deviceset="DIODE" device="SOD-123F"/>
 <part name="SUPPLY3" library="SparkFun-Aesthetics" deviceset="VCC" device=""/>
-<part name="JP3" library="SparkFun-Connectors" deviceset="M05X2" device="PTH"/>
-<part name="JP6" library="SparkFun-Connectors" deviceset="M05X2" device="PTH"/>
+<part name="JP3" library="SparkFun-Connectors" deviceset="M05X2" device="SHD" value="M05X2SHD"/>
+<part name="JP6" library="SparkFun-Connectors" deviceset="M05X2" device="SHD" value="M05X2SHD"/>
 <part name="SJ4" library="SparkFun-Retired" deviceset="SOLDERJUMPER" device="TRACE"/>
 <part name="SUPPLY4" library="SparkFun-Aesthetics" deviceset="VCC" device=""/>

Commit message: layout and working on silks
Parts:
- J2: value HEADER-M26 -> ACCESSORY
Connections:
- removed net N$8: IC3.VCC@14, IC3.VCC@34
- net VCCIC: now also IC3.VCC@14, IC3.VCC@34
Changed lines of the file:
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@@
 <part name="SJ2" library="SparkFun-Passives" deviceset="SOLDERJUMPER" device="NO"/>
 <part name="SJ3" library="SparkFun-Passives" deviceset="SOLDERJUMPER" device="TRACE"/>
-<part name="J2" library="digits" deviceset="HEADER-M26" device=""/>
+<part name="J2" library="digits" deviceset="HEADER-M26" device="" value="ACCESSORY"/>
 <part name="SUPPLY15" library="SparkFun-Aesthetics" deviceset="VCC" device="" value="VCC"/>
 <part name="GND16" library="SparkFun-Aesthetics" deviceset="GND" device=""/>
@@
 </segment>
 </net>
-<net name="N$8" class="0">
-<segment>
-<pinref part="IC3" gate="G$1" pin="VCC@14"/>
-<wire x1="307.34" y1="58.42" x2="292.1" y2="58.42" width="0.1524" layer="91"/>
-<pinref part="IC3" gate="G$1" pin="VCC@34"/>
-<wire x1="307.34" y1="55.88" x2="292.1" y2="55.88" width="0.1524" layer="91"/>
-<wire x1="292.1" y1="55.88" x2="292.1" y2="58.42" width="0.1524" layer="91"/>
-</segment>
-</net>
 <net name="VCCIC" class="0">
 <segment>
@@
 <wire x1="279.4" y1="58.42" x2="292.1" y2="58.42" width="0.1524" layer="91"/>
 <pinref part="R6" gate="G$1" pin="2"/>
-<wire x1="292.1" y1="58.42" x2="294.64" y2="58.42" width="0.1524" layer="91"/>
 <wire x1="294.64" y1="60.96" x2="292.1" y2="60.96" width="0.1524" layer="91"/>
 <wire x1="292.1" y1="60.96" x2="292.1" y2="58.42" width="0.1524" layer="91"/>
+<junction x="279.4" y="58.42"/>
+<pinref part="IC3" gate="G$1" pin="VCC@34"/>
+<wire x1="307.34" y1="55.88" x2="292.1" y2="55.88" width="0.1524" layer="91"/>
+<wire x1="292.1" y1="55.88" x2="292.1" y2="58.42" width="0.1524" layer="91"/>
+<pinref part="IC3" gate="G$1" pin="VCC@14"/>
+<wire x1="307.34" y1="58.42" x2="292.1" y2="58.42" width="0.1524" layer="91"/>
 <junction x="292.1" y="58.42"/>
-<junction x="279.4" y="58.42"/>
-</segment>
-<segment>
+</segment>
+<segment>
