File: digits.sch (EAGLE design)
At the start: 48 parts, among them IC1 STP16CP05 / STP16CPC26, IC2 STP16CP05 / STP16CPC26, IC3 ATMEGA32U4QFN, IC4 ATMEGA32U4TQFP-44, J1 POWER_JACKPTH_LOCK, J2 ACCESSORY, X1 CRYSTALHC49

Commit message: layout
Parts:
- JP4: value Bluefruit LE -> Adafruit Bluefruit LE
Connections:
- net PD0: now also J2.11; no longer J2.9
- net PD1: now also J2.9; no longer J2.11
Changed lines of the file:
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@@
 <part name="R8" library="SparkFun-Resistors" deviceset="RESISTOR" device="0805-RES" value="910R"/>
 <part name="GND14" library="SparkFun-Aesthetics" deviceset="GND" device=""/>
-<part name="JP4" library="SparkFun-Connectors" deviceset="M10" device="LOCK" value="Bluefruit LE"/>
+<part name="JP4" library="SparkFun-Connectors" deviceset="M10" device="LOCK" value="Adafruit Bluefruit LE"/>
 <part name="GND23" library="SparkFun-Aesthetics" deviceset="GND" device=""/>
 <part name="SUPPLY9" library="SparkFun-Aesthetics" deviceset="VCC" device=""/>
@@
 </segment>
 <segment>
+<pinref part="JP3" gate="G$1" pin="8"/>
+<wire x1="20.32" y1="35.56" x2="22.86" y2="35.56" width="0.1524" layer="91"/>
+<label x="22.86" y="35.56" size="1.4224" layer="95" xref="yes"/>
+</segment>
+<segment>
+<pinref part="JP6" gate="G$1" pin="3"/>
+<wire x1="60.96" y1="35.56" x2="63.5" y2="35.56" width="0.1524" layer="91"/>
+<label x="63.5" y="35.56" size="1.4224" layer="95" xref="yes"/>
+</segment>
+<segment>
+<wire x1="492.76" y1="27.94" x2="490.22" y2="27.94" width="0.1524" layer="91"/>
+<label x="490.22" y="27.94" size="1.4224" layer="95" rot="R180" xref="yes"/>
+<pinref part="J2" gate="G$1" pin="9"/>
+</segment>
+</net>
+<net name="PD0" class="0">
+<segment>
+<pinref part="IC4" gate="G$1" pin="PD0(SCL)"/>
+<wire x1="434.34" y1="30.48" x2="436.88" y2="30.48" width="0.1524" layer="91"/>
+<label x="436.88" y="30.48" size="1.4224" layer="95" xref="yes"/>
+</segment>
+<segment>
+<pinref part="IC3" gate="G$1" pin="PD0(SCL)"/>
+<wire x1="342.9" y1="30.48" x2="345.44" y2="30.48" width="0.1524" layer="91"/>
+<label x="345.44" y="30.48" size="1.4224" layer="95" xref="yes"/>
+</segment>
+<segment>
+<pinref part="JP3" gate="G$1" pin="7"/>
+<wire x1="5.08" y1="35.56" x2="2.54" y2="35.56" width="0.1524" layer="91"/>
+<label x="2.54" y="35.56" size="1.4224" layer="95" rot="R180" xref="yes"/>
+</segment>
+<segment>
+<pinref part="JP6" gate="G$1" pin="4"/>
+<wire x1="45.72" y1="35.56" x2="43.18" y2="35.56" width="0.1524" layer="91"/>
+<label x="43.18" y="35.56" size="1.4224" layer="95" rot="R180" xref="yes"/>
+</segment>
+<segment>
 <wire x1="492.76" y1="25.4" x2="490.22" y2="25.4" width="0.1524" layer="91"/>
 <label x="490.22" y="25.4" size="1.4224" layer="95" rot="R180" xref="yes"/>
 <pinref part="J2" gate="G$1" pin="11"/>
 </segment>
-<segment>
-<pinref part="JP3" gate="G$1" pin="8"/>
-<wire x1="20.32" y1="35.56" x2="22.86" y2="35.56" width="0.1524" layer="91"/>
-<label x="22.86" y="35.56" size="1.4224" layer="95" xref="yes"/>
-</segment>
-<segment>
-<pinref part="JP6" gate="G$1" pin="3"/>
-<wire x1="60.96" y1="35.56" x2="63.5" y2="35.56" width="0.1524" layer="91"/>
-<label x="63.5" y="35.56" size="1.4224" layer="95" xref="yes"/>
-</segment>
-</net>
-<net name="PD0" class="0">
-<segment>
-<pinref part="IC4" gate="G$1" pin="PD0(SCL)"/>
-<wire x1="434.34" y1="30.48" x2="436.88" y2="30.48" width="0.1524" layer="91"/>
-<label x="436.88" y="30.48" size="1.4224" layer="95" xref="yes"/>
-</segment>
-<segment>
-<pinref part="IC3" gate="G$1" pin="PD0(SCL)"/>
-<wire x1="342.9" y1="30.48" x2="345.44" y2="30.48" width="0.1524" layer="91"/>
-<label x="345.44" y="30.48" size="1.4224" layer="95" xref="yes"/>
-</segment>
-<segment>
-<wire x1="492.76" y1="27.94" x2="490.22" y2="27.94" width="0.1524" layer="91"/>
-<label x="490.22" y="27.94" size="1.4224" layer="95" rot="R180" xref="yes"/>
-<pinref part="J2" gate="G$1" pin="9"/>
-</segment>
-<segment>
-<pinref part="JP3" gate="G$1" pin="7"/>
-<wire x1="5.08" y1="35.56" x2="2.54" y2="35.56" width="0.1524" layer="91"/>
-<label x="2.54" y="35.56" size="1.4224" layer="95" rot="R180" xref="yes"/>
-</segment>
-<segment>
-<pinref part="JP6" gate="G$1" pin="4"/>
-<wire x1="45.72" y1="35.56" x2="43.18" y2="35.56" width="0.1524" layer="91"/>
-<label x="43.18" y="35.56" size="1.4224" layer="95" rot="R180" xref="yes"/>
-</segment>
-</net>
+</net>

Commit message: layout, added diode
Parts:
- added D2: (no value), SparkFun-DiscreteSemi:DIODESOD
- D1: value DIODESOD-123F -> (none); device digits:DIODESOD-123F -> SparkFun-DiscreteSemi:DIODESOD
Connections:
- new net N$6: D2.A, J1.PWR
- net VCC: now also D2.C; no longer J1.PWR
Changed lines of the file:
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@@
 <part name="T5" library="zetex" deviceset="PMOSSOT23" device=""/>
 <part name="SUPPLY21" library="SparkFun-Aesthetics" deviceset="VCC" device="" value="VCC"/>
-<part name="D1" library="digits" deviceset="DIODE" device="SOD-123F"/>
+<part name="D1" library="SparkFun-DiscreteSemi" deviceset="DIODE" device="SOD"/>
 <part name="SUPPLY3" library="SparkFun-Aesthetics" deviceset="VCC" device=""/>
 <part name="JP3" library="SparkFun-Connectors" deviceset="M05X2" device="SHD" value="M05X2SHD"/>
@@
 <part name="SJ4" library="SparkFun-Retired" deviceset="SOLDERJUMPER" device="TRACE"/>
 <part name="SUPPLY4" library="SparkFun-Aesthetics" deviceset="VCC" device=""/>
+<part name="D2" library="SparkFun-DiscreteSemi" deviceset="DIODE" device="SOD"/>
 </parts>
 <sheets>
@@
 <instance part="SJ4" gate="1" x="279.4" y="73.66" rot="R90"/>
 <instance part="SUPPLY4" gate="G$1" x="279.4" y="83.82"/>
+<instance part="D2" gate="G$1" x="281.94" y="-40.64"/>
 </instances>
 <busses>
@@
 </segment>
 <segment>
-<pinref part="J1" gate="G$1" pin="PWR"/>
-<pinref part="SUPPLY15" gate="G$1" pin="VCC"/>
-<wire x1="271.78" y1="-40.64" x2="292.1" y2="-40.64" width="0.1524" layer="91"/>
-<wire x1="292.1" y1="-40.64" x2="292.1" y2="-38.1" width="0.1524" layer="91"/>
-</segment>
-<segment>
 <pinref part="T1" gate="A" pin="D"/>
 <pinref part="SUPPLY17" gate="G$1" pin="VCC"/>
@@
 <wire x1="60.96" y1="43.18" x2="63.5" y2="43.18" width="0.1524" layer="91"/>
 <label x="63.5" y="43.18" size="1.4224" layer="95" xref="yes"/>
+</segment>
+<segment>
+<pinref part="D2" gate="G$1" pin="C"/>
+<pinref part="SUPPLY15" gate="G$1" pin="VCC"/>
+<wire x1="284.48" y1="-40.64" x2="292.1" y2="-40.64" width="0.1524" layer="91"/>
+<wire x1="292.1" y1="-40.64" x2="292.1" y2="-38.1" width="0.1524" layer="91"/>
 </segment>
 </net>
@@
 </segment>
 </net>
+<net name="N$6" class="0">
+<segment>
+<pinref part="J1" gate="G$1" pin="PWR"/>
+<pinref part="D2" gate="G$1" pin="A"/>
+<wire x1="271.78" y1="-40.64" x2="279.4" y2="-40.64" width="0.1524" layer="91"/>
+</segment>
+</net>

Commit message: finished BOM
Parts:
- C1, C2, C7, C8, C9: PARTNO (none) -> C0805C104K5RACTU
- C3, C6: PARTNO (none) -> CL21B105KBFNNNE
- C4, C5: PARTNO (none) -> C0805C220J5GACTU
- D1, D2: value (none) -> PMEG3030EP; device SparkFun-DiscreteSemi:DIODESOD -> digits:DIODESOD-128; PARTNO (none) -> PMEG3030EP-115
- IC1, IC2: PARTNO (none) -> STP16CPC26MTR
- IC3: PARTNO (none) -> ATMEGA32U4-MUR
- IC4: PARTNO (none) -> ATMEGA32U4-AU
- J1: PARTNO (none) -> PJ-202A
- J2: PARTNO (none) -> SFH11-PBPC-D13-ST-BK
- JP1: PARTNO (none) -> M20-9980346
- JP2: PARTNO (none) -> 690-005-299-043
- JP3, JP6: PARTNO (none) -> 302-S101
- L1: PARTNO (none) -> CIM21J601NE
- LED1: PARTNO (none) -> LG R971-KN-1
- R1: PARTNO (none) -> RC0805FR-07390RL
- R2, R8: PARTNO (none) -> MCR10ERTF9100
- R3, R4: PARTNO (none) -> RC0805FR-0722RL
- R5: PARTNO (none) -> RC0805FR-071ML
- R6: PARTNO (none) -> RC0805JR-0710KL
- SJ1, SJ2, SJ3, SJ4: BOM (none) -> EXCLUDE
- T1, T2, T3, T4, T5: PARTNO (none) -> FDN352AP
- X1: PARTNO (none) -> 9C-16.000MAAJ-T
- Z1, Z2: PARTNO (none) -> CG0603MLC-05E
