File: Hardware/alpha.brd (EAGLE design)
At the start: 240.8 x 81 mm, 67 parts, among them IC1 STP16CP05 / STP16CPC26, IC2 STP16CP05 / STP16CPC26, IC3 ATMEGA32U4QFN, IC4 ATMEGA32U4TQFP-44, IC5 CHRONODOT, IC6 7805DT, J1 POWER_JACKPTH_LOCK, J2 ACCESSORY, X1 CRYSTALHC49

Commit message: added Alpha text
Other:
- board text added: "Alpha"
- board text added: "LED Display"

Commit message: old changes from laptop, double check
Parts:
- removed JP4: (no value), SparkFun-Connectors:1X03_LOCK
- added IC7: Pololu Step-Up, alpha:1X03_LOCK
- moved D3 4.40 mm to (47.8, 22.4)
- turned JP6 to 0 degrees
Connections:
- net GND: now also IC7.2; no longer JP4.2
- net N$13: now also IC7.3; no longer JP4.3
- net VCC5V: now also IC7.1; no longer JP4.1
Routing:
- net VCC5V: track 474.7 -> 497.0 mm
- net D7: track 351.1 -> 335.2 mm, vias 12 -> 11
- net VCC9V: track 375.8 -> 360.3 mm, vias 14 -> 13
- net ROW1: track 96.4 -> 107.1 mm
- net D1/TX: track 236.3 -> 246.6 mm
- net N$13: track 3.36 -> 12.5 mm
- net D0/RX: track 241.4 -> 236.4 mm, vias 8 -> 10
- net BLANK: track 171.6 -> 174.2 mm
- net D2/SDA: track 354.9 -> 356.7 mm
- net N$16: track 25.6 -> 23.8 mm
- net D10: track 137.5 -> 135.8 mm
- net COL-DP: track 268.6 -> 270.1 mm
- net D3/SCL: track 347.9 -> 349.4 mm, vias 8 -> 9
- net D9: track 176.6 -> 175.2 mm
- net D11: track 123.2 -> 121.8 mm
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Other:
- board text added: "Rev B 2014 (TAPR OHL)"
- board text removed: "Rev B 2014 (CC BY-SA 3.0)"
