File: Hardware/alpha.sch (EAGLE design)
At the start: 67 parts, among them IC1 STP16CP05 / STP16CPC26, IC2 STP16CP05 / STP16CPC26, IC3 ATMEGA32U4QFN, IC4 ATMEGA32U4TQFP-44, IC5 CHRONODOT, IC6 7805DT, J1 POWER_JACKPTH_LOCK, J2 ACCESSORY, X1 CRYSTALHC49

Commit message: old changes from laptop, double check
Parts:
- removed JP4: (no value), SparkFun-Connectors:M03LOCK
- added IC7: Pololu Step-Up, alpha:POLOLU_REG
Connections:
- net GND: now also IC7.GND; no longer JP4.2
- net N$13: now also IC7.VOUT; no longer JP4.3
- net VCC5V: now also IC7.VIN; no longer JP4.1
Other:
- moved on the sheet: D3
Changed lines of the file:
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@@
 <?xml version="1.0" encoding="utf-8"?>
 <!DOCTYPE eagle SYSTEM "eagle.dtd">
-<eagle version="6.6.0">
+<eagle version="6.4">
 <drawing>
 <settings>
@@
 </part>
 <part name="SUPPLY9" library="SparkFun-Aesthetics" deviceset="VCC" device="" value="VCC5v"/>
-<part name="JP4" library="SparkFun-Connectors" deviceset="M03" device="LOCK"/>
 <part name="SUPPLY6" library="SparkFun-Aesthetics" deviceset="VCC" device="" value="VCC9v"/>
 <part name="GND19" library="SparkFun-Aesthetics" deviceset="GND" device=""/>
@@
 <part name="R19" library="SparkFun-Resistors" deviceset="RESISTOR" device="0805-RES" value="10k"/>
 <part name="SUPPLY12" library="SparkFun-Aesthetics" deviceset="VCC" device="" value="VCC5v"/>
+<part name="IC7" library="alpha" deviceset="POLOLU_REG" device="" value="Pololu Step-Up"/>
 </parts>
 <sheets>
@@
 </instance>
 <instance part="SUPPLY9" gate="G$1" x="55.88" y="160.02"/>
-<instance part="JP4" gate="G$1" x="68.58" y="167.64"/>
-<instance part="SUPPLY6" gate="G$1" x="86.36" y="172.72"/>
-<instance part="GND19" gate="1" x="91.44" y="162.56"/>
-<instance part="SUPPLY7" gate="G$1" x="83.82" y="160.02"/>
-<instance part="D3" gate="G$1" x="81.28" y="170.18">
-<attribute name="PARTNO" x="81.28" y="170.18" size="1.778" layer="96" display="off"/>
+<instance part="SUPPLY6" gate="G$1" x="104.14" y="182.88"/>
+<instance part="GND19" gate="1" x="78.74" y="165.1"/>
+<instance part="SUPPLY7" gate="G$1" x="60.96" y="185.42"/>
+<instance part="D3" gate="G$1" x="99.06" y="180.34">
+<attribute name="PARTNO" x="99.06" y="180.34" size="1.778" layer="96" display="off"/>
 </instance>
 <instance part="R13" gate="G$1" x="43.18" y="231.14">
@@
 <instance part="R19" gate="G$1" x="129.54" y="180.34" rot="R90"/>
 <instance part="SUPPLY12" gate="G$1" x="129.54" y="187.96"/>
+<instance part="IC7" gate="G$1" x="78.74" y="177.8"/>
 </instances>
 <busses>
@@
 </segment>
 <segment>
-<pinref part="JP4" gate="G$1" pin="2"/>
-<pinref part="GND19" gate="1" pin="GND"/>
-<wire x1="76.2" y1="167.64" x2="91.44" y2="167.64" width="0.1524" layer="91"/>
-<wire x1="91.44" y1="167.64" x2="91.44" y2="165.1" width="0.1524" layer="91"/>
-</segment>
-<segment>
 <pinref part="IC5" gate="G$1" pin="GND"/>
 <pinref part="GND20" gate="1" pin="GND"/>
 <wire x1="360.68" y1="60.96" x2="358.14" y2="60.96" width="0.1524" layer="91"/>
 <wire x1="358.14" y1="60.96" x2="358.14" y2="58.42" width="0.1524" layer="91"/>
+</segment>
+<segment>
+<pinref part="IC7" gate="G$1" pin="GND"/>
+<pinref part="GND19" gate="1" pin="GND"/>
+<wire x1="78.74" y1="170.18" x2="78.74" y2="167.64" width="0.1524" layer="91"/>
 </segment>
 </net>
@@
 </segment>
 <segment>
-<pinref part="JP4" gate="G$1" pin="1"/>
-<wire x1="76.2" y1="165.1" x2="78.74" y2="165.1" width="0.1524" layer="91"/>
-<wire x1="78.74" y1="165.1" x2="78.74" y2="157.48" width="0.1524" layer="91"/>
-<pinref part="SUPPLY7" gate="G$1" pin="VCC"/>
-<wire x1="78.74" y1="157.48" x2="83.82" y2="157.48" width="0.1524" layer="91"/>
-<wire x1="83.82" y1="157.48" x2="83.82" y2="160.02" width="0.1524" layer="91"/>
-</segment>
-<segment>
 <pinref part="SUPPLY11" gate="G$1" pin="VCC"/>
 <pinref part="R18" gate="G$1" pin="1"/>
@@
 <pinref part="R19" gate="G$1" pin="2"/>
 <wire x1="129.54" y1="187.96" x2="129.54" y2="185.42" width="0.1524" layer="91"/>
+</segment>
+<segment>
+<pinref part="IC7" gate="G$1" pin="VIN"/>
+<pinref part="SUPPLY7" gate="G$1" pin="VCC"/>
+<wire x1="63.5" y1="180.34" x2="60.96" y2="180.34" width="0.1524" layer="91"/>
+<wire x1="60.96" y1="180.34" x2="60.96" y2="185.42" width="0.1524" layer="91"/>
 </segment>
 </net>
@@
 <pinref part="D3" gate="G$1" pin="C"/>
 <pinref part="SUPPLY6" gate="G$1" pin="VCC"/>
-<wire x1="83.82" y1="170.18" x2="86.36" y2="170.18" width="0.1524" layer="91"/>
-<wire x1="86.36" y1="170.18" x2="86.36" y2="172.72" width="0.1524" layer="91"/>
+<wire x1="101.6" y1="180.34" x2="104.14" y2="180.34" width="0.1524" layer="91"/>
+<wire x1="104.14" y1="180.34" x2="104.14" y2="182.88" width="0.1524" layer="91"/>
 </segment>
 <segment>
@@
 <wire x1="114.3" y1="50.8" x2="116.84" y2="50.8" width="0.1524" layer="91"/>
 <label x="116.84" y="50.8" size="1.4224" layer="95" xref="yes"/>
-</segment>
-</net>
-<net name="N$13" class="0">
-<segment>
-<pinref part="JP4" gate="G$1" pin="3"/>
-<pinref part="D3" gate="G$1" pin="A"/>
-<wire x1="76.2" y1="170.18" x2="78.74" y2="170.18" width="0.1524" layer="91"/>
 </segment>
 </net>
@@
 </segment>
 </net>
+<net name="N$13" class="0">
+<segment>
+<pinref part="D3" gate="G$1" pin="A"/>
+<pinref part="IC7" gate="G$1" pin="VOUT"/>
+<wire x1="96.52" y1="180.34" x2="93.98" y2="180.34" width="0.1524" layer="91"/>
+</segment>
+</net>
